Commit message: changing urdf physics

File: fellahbot_description/urdf/constants.xacro (robot description, xacro)
@@ -9,4 +9,5 @@
 	<!-- Chassis properties -->
 	<xacro:property name="chassis_height" value="0.311"/>
+	<!--xacro:property name="chassis_height" value="0.470"/-->
 	<!--xacro:property name="chassis_height" value="0.411"/-->
 	<xacro:property name="chassis_length" value="1.150"/>

File: fellahbot_description/urdf/fellahbot.urdf.xacro (robot description, xacro)
@@ -135,5 +135,5 @@
       <material name="yellow"/>
     </collision>
-    <xacro:default_inertial mass="1"/>
+    <xacro:solid_cylinder_inertial rpy="0 0 0" xyz="0.319 0.0 0.0" mass="1" radius="0.05" length="0.03" />
   </link>
   <joint name="steer_joint" type="revolute">
@@ -141,5 +141,5 @@
     <child link="steer_link"/>
     <axis xyz="0 0 1"/>
-    <limit lower="-${math_pi_over_6}" upper="${math_pi_over_6}" velocity="5.0" effort="10.0"/>
+    <limit lower="-${math_pi_over_6}" upper="${math_pi_over_6}" velocity="25.0" effort="50.0"/>
     <origin xyz="0.319 0.0 0.0"/>
   </joint>
@@ -174,5 +174,5 @@
       <material name="yellow"/>
     </collision>
-    <xacro:default_inertial mass="1"/>
+    <xacro:solid_cylinder_inertial rpy="0 0 0" xyz="-0.335 0.0 -0.192" mass="1" radius="0.03" length="0.05" />
   </link>
   <joint name="wheel_joint" type="continuous">
@@ -180,6 +180,6 @@
     <child link="wheel_link"/>
     <origin xyz="-0.335 0.0 -0.192" rpy="0 0 0"/>
-    <limit effort="10" velocity="10"/>
-    <joint_properties damping="0.01" friction="0.0"/>
+    <limit effort="150" velocity="20"/>
+    <joint_properties damping="0.2" friction="0.8"/>
   </joint>
   <!-- Transmission is important to link the joints and the controller -->

File: fellahbot_description/urdf/wheel.xacro (robot description, xacro)
@@ -25,5 +25,5 @@
             <child link="front_${prefix}_steer"/>
             <axis xyz="0 0 1"/>
-            <limit lower="-${math_pi_over_6}" upper="${math_pi_over_6}" velocity="5.0" effort="10.0"/>
+            <limit lower="-${math_pi_over_6}" upper="${math_pi_over_6}" velocity="25.0" effort="50"/>
             <origin xyz="0.319 ${(reflect * 0.175)} 0.0"/>
         </joint>
@@ -31,10 +31,10 @@
             <type>transmission_interface/SimpleTransmission</type>
             <joint name="front_${prefix}_steer_joint">
-                <hardwareInterface>hardware_interface/PositionJointInterface</hardwareInterface>
+                <hardwareInterface>PositionJointInterface</hardwareInterface>
             </joint>
             <actuator name="front_${prefix}_steer_motor">
                 <mechanicalReduction>1.0</mechanicalReduction>
                 <motorTorqueConstant>1.0</motorTorqueConstant>
-                <hardwareInterface>hardware_interface/PositionJointInterface</hardwareInterface>
+                <hardwareInterface>PositionJointInterface</hardwareInterface>
             </actuator>
         </transmission>
@@ -58,16 +58,16 @@
             <axis xyz="0 1 0"/>
             <origin xyz="0.0 0.0 -0.192" rpy="0 0 0"/>
-            <limit effort="10" velocity="10"/>
-            <joint_properties damping="0.01" friction="0.0"/>
+            <limit effort="150" velocity="20"/>
+            <joint_properties damping="0.2" friction="0.8"/>
         </joint>
         <transmission name="front_${prefix}_wheel_transmission">
             <type>transmission_interface/SimpleTransmission</type>
             <joint name="front_${prefix}_wheel_joint">
-                <hardwareInterface>hardware_interface/VelocityJointInterface</hardwareInterface>
+                <hardwareInterface>VelocityJointInterface</hardwareInterface>
             </joint>
             <actuator name="front_${prefix}_motor">
                 <mechanicalReduction>1.0</mechanicalReduction>
                 <motorTorqueConstant>1.0</motorTorqueConstant>
-                <hardwareInterface>hardware_interface/VelocityJointInterface</hardwareInterface>
+                <hardwareInterface>VelocityJointInterface</hardwareInterface>
             </actuator>
         </transmission>
@@ -78,5 +78,5 @@
         <xacro:property name="pos_z_joint" value="-${chassis_to_ground - wheel_radius}"/>
         <link name="rear_${prefix}_wheel">
-        <visual>
+            <visual>
                 <geometry>
                     <mesh filename="package://fellahbot_description/meshes/Fellahbot_DAE/Parts/Geared_Hub_Motor-Fusion001.dae"/>
@@ -96,16 +96,16 @@
             <axis xyz="0 1 0"/>
             <origin xyz="-0.335 ${(reflect * 0.17523)} -0.192" rpy="0 0 0"/>
-            <limit effort="10" velocity="10"/>
-            <joint_properties damping="0.01" friction="0.0"/>
+            <limit effort="150" velocity="20"/>
+            <joint_properties damping="0.2" friction="0.8"/>
         </joint>
         <transmission name="rear_${prefix}_wheel_transmission">
             <type>transmission_interface/SimpleTransmission</type>
             <joint name="rear_${prefix}_wheel_joint">
-                <hardwareInterface>hardware_interface/VelocityJointInterface</hardwareInterface>
+                <hardwareInterface>VelocityJointInterface</hardwareInterface>
             </joint>
             <actuator name="rear_${prefix}_motor">
                 <mechanicalReduction>1.0</mechanicalReduction>
                 <motorTorqueConstant>1.0</motorTorqueConstant>
-                <hardwareInterface>hardware_interface/VelocityJointInterface</hardwareInterface>
+                <hardwareInterface>VelocityJointInterface</hardwareInterface>
             </actuator>
         </transmission>

Commit message: adding inertial and physics parameters

File: fellahbot_description/urdf/constants.xacro (robot description, xacro)
@@ -6,5 +6,6 @@
 	<xacro:property name="math_pi_over_2" value="1.5707963267948966" />
 	<xacro:property name="math_pi_over_4" value="0.785398163397448" />
-	<xacro:property name="math_pi_over_6" value="${(PI/(6.0))}" />
+	<xacro:property name="math_pi_over_6" value="${(math_pi/(6.0))}" />
+	<xacro:property name="math_pi_over_6_29" value="0.51" />
 	<!-- Chassis properties -->
 	<xacro:property name="chassis_height" value="0.311"/>

File: fellahbot_description/urdf/fellahbot.urdf.xacro (robot description, xacro)
@@ -21,5 +21,5 @@
       </geometry>
     </collision>
-    <xacro:default_inertial mass="50"/>
+    <xacro:solid_cuboid_inertial rpy="0 0 0" xyz="0.0 0.0 0.359" mass="${chassis_mass}" x="${chassis_length}" y="${chassis_width}" z="0.411" />
   </link>
   <joint name="base_robot" type="fixed">
@@ -135,5 +135,5 @@
       <material name="yellow"/>
     </collision>
-    <xacro:solid_cylinder_inertial rpy="0 0 0" xyz="0.319 0.0 0.0" mass="1" radius="0.05" length="0.03" />
+    <xacro:solid_cylinder_inertial rpy="0 0 0" xyz="0.319 0.0 0.0" mass="6" radius="0.05" length="0.03" />
   </link>
   <joint name="steer_joint" type="revolute">
@@ -141,21 +141,26 @@
     <child link="steer_link"/>
     <axis xyz="0 0 1"/>
-    <limit lower="-${math_pi_over_6}" upper="${math_pi_over_6}" velocity="25.0" effort="50.0"/>
+    <limit lower="${-math_pi_over_6_29}" upper="${math_pi_over_6}" velocity="50.0" effort="100.0"/>
     <origin xyz="0.319 0.0 0.0"/>
   </joint>
   <!-- Transmission is important to link the joints and the controller -->
-   <transmission name="steer_joint_trans">
-      <type>transmission_interface/SimpleTransmission</type>
-      <actuator name="steer_joint_motor">
-        <mechanicalReduction>1.0</mechanicalReduction>
-        <motorTorqueConstant>1.0</motorTorqueConstant>
-        <hardwareInterface>hardware_interface/PositionJointInterface</hardwareInterface>
-      </actuator>
-      <joint name="steer_joint">
-        <hardwareInterface>hardware_interface/PositionJointInterface</hardwareInterface>
-      </joint>
-    </transmission>
+  <transmission name="steer_joint_trans">
+    <type>transmission_interface/SimpleTransmission</type>
+    <actuator name="steer_joint_motor">
+      <mechanicalReduction>1.0</mechanicalReduction>
+      <motorTorqueConstant>1.0</motorTorqueConstant>
+      <hardwareInterface>hardware_interface/PositionJointInterface</hardwareInterface>
+    </actuator>
+    <joint name="steer_joint">
+      <hardwareInterface>hardware_interface/PositionJointInterface</hardwareInterface>
+    </joint>
+  </transmission>
   <gazebo reference="steer_link">
     <material>Gazebo/Yellow</material>
+    <mu1 value="1.0"/>
+    <mu2 value="1.0"/>
+    <kp value="10000000.0" />
+    <kd value="1.0" />
+    <fdir1 value="1 0 0"/>
   </gazebo>
   <link name="wheel_link">
@@ -174,5 +179,5 @@
       <material name="yellow"/>
     </collision>
-    <xacro:solid_cylinder_inertial rpy="0 0 0" xyz="-0.335 0.0 -0.192" mass="1" radius="0.03" length="0.05" />
+    <xacro:solid_cylinder_inertial rpy="0 0 0" xyz="-0.335 0.0 -0.192" mass="6" radius="0.03" length="0.05" />
   </link>
   <joint name="wheel_joint" type="continuous">
@@ -181,5 +186,5 @@
     <origin xyz="-0.335 0.0 -0.192" rpy="0 0 0"/>
     <limit effort="150" velocity="20"/>
-    <joint_properties damping="0.2" friction="0.8"/>
+    <joint_properties damping="1.0" friction="1.0"/>
   </joint>
   <!-- Transmission is important to link the joints and the controller -->
@@ -197,4 +202,9 @@
   <gazebo reference="wheel_link">
     <material>Gazebo/Yellow</material>
+    <mu1 value="1.0"/>
+    <mu2 value="1.0"/>
+    <kp value="10000000.0" />
+    <kd value="1.0" />
+    <fdir1 value="1 0 0"/>
   </gazebo>
 </robot>

File: fellahbot_description/urdf/plugin.gazebo.xacro (robot description, xacro)
@@ -13,4 +13,6 @@
   </gazebo>
   <gazebo reference="camera">
+    <mu1>0.2</mu1>
+    <mu2>0.2</mu2>
     <material>Gazebo/Red</material>
     <sensor name="camera1" type="camera">

File: fellahbot_description/urdf/wheel.xacro (robot description, xacro)
@@ -25,5 +25,5 @@
             <child link="front_${prefix}_steer"/>
             <axis xyz="0 0 1"/>
-            <limit lower="-${math_pi_over_6}" upper="${math_pi_over_6}" velocity="25.0" effort="50"/>
+            <limit lower="${-math_pi_over_6_29}" upper="${math_pi_over_6}" velocity="50.0" effort="100"/>
             <origin xyz="0.319 ${(reflect * 0.175)} 0.0"/>
         </joint>
@@ -31,10 +31,10 @@
             <type>transmission_interface/SimpleTransmission</type>
             <joint name="front_${prefix}_steer_joint">
-                <hardwareInterface>PositionJointInterface</hardwareInterface>
+                <hardwareInterface>hardware_interface/PositionJointInterface</hardwareInterface>
             </joint>
             <actuator name="front_${prefix}_steer_motor">
                 <mechanicalReduction>1.0</mechanicalReduction>
                 <motorTorqueConstant>1.0</motorTorqueConstant>
-                <hardwareInterface>PositionJointInterface</hardwareInterface>
+                <hardwareInterface>hardware_interface/PositionJointInterface</hardwareInterface>
             </actuator>
         </transmission>
@@ -59,17 +59,24 @@
             <origin xyz="0.0 0.0 -0.192" rpy="0 0 0"/>
             <limit effort="150" velocity="20"/>
-            <joint_properties damping="0.2" friction="0.8"/>
+            <joint_properties damping="1.0" friction="1.0"/>
         </joint>
         <transmission name="front_${prefix}_wheel_transmission">
             <type>transmission_interface/SimpleTransmission</type>
             <joint name="front_${prefix}_wheel_joint">
-                <hardwareInterface>VelocityJointInterface</hardwareInterface>
+                <hardwareInterface>hardware_interface/VelocityJointInterface</hardwareInterface>
             </joint>
             <actuator name="front_${prefix}_motor">
                 <mechanicalReduction>1.0</mechanicalReduction>
                 <motorTorqueConstant>1.0</motorTorqueConstant>
-                <hardwareInterface>VelocityJointInterface</hardwareInterface>
+                <hardwareInterface>hardware_interface/VelocityJointInterface</hardwareInterface>
             </actuator>
         </transmission>
+        <gazebo reference="front_${prefix}_wheel">
+            <mu1 value="1.0"/>
+			<mu2 value="1.0"/>
+			<kp value="10000000.0" />
+			<kd value="1.0" />
+			<fdir1 value="1 0 0"/>
+        </gazebo>
     </xacro:macro>
     <xacro:macro name="rear_wheel" params="prefix parent reflect ">
@@ -97,17 +104,24 @@
             <origin xyz="-0.335 ${(reflect * 0.17523)} -0.192" rpy="0 0 0"/>
             <limit effort="150" velocity="20"/>
-            <joint_properties damping="0.2" friction="0.8"/>
+            <joint_properties damping="1.0" friction="1.0"/>
         </joint>
         <transmission name="rear_${prefix}_wheel_transmission">
             <type>transmission_interface/SimpleTransmission</type>
             <joint name="rear_${prefix}_wheel_joint">
-                <hardwareInterface>VelocityJointInterface</hardwareInterface>
+                <hardwareInterface>hardware_interface/VelocityJointInterface</hardwareInterface>
             </joint>
             <actuator name="rear_${prefix}_motor">
                 <mechanicalReduction>1.0</mechanicalReduction>
                 <motorTorqueConstant>1.0</motorTorqueConstant>
-                <hardwareInterface>VelocityJointInterface</hardwareInterface>
+                <hardwareInterface>hardware_interface/VelocityJointInterface</hardwareInterface>
             </actuator>
         </transmission>
+        <gazebo reference="rear_${prefix}_wheel">
+            <mu1 value="1.0"/>
+			<mu2 value="1.0"/>
+			<kp value="10000000.0" />
+			<kd value="1.0" />
+			<fdir1 value="1 0 0"/>
+        </gazebo>
     </xacro:macro>
 </robot>
