Commit message: create fellahbot_gazebo pkg and urdf file revision

File: fellahbot_description/urdf/fellahbot.urdf.xacro (robot description, xacro)
@@ -29,5 +29,5 @@
   </joint>
   <!-- lidar link -->
-  <link name="lidar">
+  <link name="laser">
     <visual>
       <geometry>
@@ -45,5 +45,5 @@
   <joint name="base_lidar" type="fixed">
     <parent link="chassis"/>
-    <child link="lidar"/>
+    <child link="laser"/>
     <origin xyz="0.455 0.0 -0.028"/>
   </joint>
@@ -126,6 +126,6 @@
       <type>transmission_interface/SimpleTransmission</type>
       <actuator name="steer_joint_motor">
-        <mechanicalReduction>1</mechanicalReduction>
-        <motorTorqueConstant>1.o</motorTorqueConstant>
+        <mechanicalReduction>1.0</mechanicalReduction>
+        <motorTorqueConstant>1.0</motorTorqueConstant>
         <hardwareInterface>hardware_interface/PositionJointInterface</hardwareInterface>
       </actuator>
@@ -169,5 +169,5 @@
     <actuator name="wheel_joint_motor">
       <mechanicalReduction>1.0</mechanicalReduction>
-      <motorTorqueConstant>1.o</motorTorqueConstant>
+      <motorTorqueConstant>1.0</motorTorqueConstant>
       <hardwareInterface>hardware_interface/VelocityJointInterface</hardwareInterface>
     </actuator>

File: fellahbot_description/urdf/plugin.gazebo.xacro (robot description, xacro)
@@ -3,15 +3,13 @@
   <xacro:include filename="$(find fellahbot_description)/urdf/constants.xacro"/>
   <xacro:include filename="$(find fellahbot_description)/urdf/inertials.xacro"/>
-   <xacro:property name="robot_namespace" value="/test1"/>
+  <xacro:property name="robot_namespace" value="/test1"/>
   <!-- ros control plugin -->
-  <xacro:macro name="ros_control">
-    <gazebo>
-      <plugin name="gazebo_ros_control" filename="libgazebo_ros_control.so">
-        <robotNamespace>${robot_namespace}</robotNamespace>
-        <robotSimType>steer_bot_hardware_gazebo/SteerBotHardwareGazebo</robotSimType>
-        <legacyModeNS>false</legacyModeNS>
-      </plugin>
-    </gazebo>
-  </xacro:macro>
+  <gazebo>
+    <plugin name="gazebo_ros_control" filename="libgazebo_ros_control.so">
+      <robotNamespace>${robot_namespace}</robotNamespace>
+      <robotSimType>steer_bot_hardware_gazebo/SteerBotHardwareGazebo</robotSimType>
+      <legacyModeNS>false</legacyModeNS>
+    </plugin>
+  </gazebo>
   <gazebo reference="camera">
     <material>Gazebo/Red</material>
@@ -47,5 +45,5 @@
   </gazebo>
   <!-- RpLidar A2 using CPU -->
-  <gazebo reference="lidar">
+  <gazebo reference="laser">
     <sensor type="ray" name="rplidar_sensor">
       <pose>0.0 0.0 0.0 0 0 0</pose>
@@ -74,9 +72,9 @@
       <plugin name="gazebo_ros_head_rplidar_controller" filename="libgazebo_ros_laser.so">
         <topicName>scan</topicName>
-        <frameName>lidar</frameName>
+        <frameName>laser</frameName>
       </plugin>
     </sensor>
   </gazebo>
-  <gazebo reference="top">
+  <gazebo reference="imu_sensor">
     <gravity>true</gravity>
     <sensor name="imu_sensor" type="imu">
@@ -84,5 +82,5 @@
       <update_rate>10</update_rate>
       <visualize>true</visualize>
-      <topic>imu</topic>
+      <topic>imu_data</topic>
       <plugin filename="libgazebo_ros_imu_sensor.so" name="imu_plugin">
         <topicName>imu</topicName>

File: fellahbot_description/urdf/wheel.xacro (robot description, xacro)
@@ -35,5 +35,5 @@
             <actuator name="front_${prefix}_steer_motor">
                 <mechanicalReduction>1.0</mechanicalReduction>
-                <motorTorqueConstant>1.o</motorTorqueConstant>
+                <motorTorqueConstant>1.0</motorTorqueConstant>
                 <hardwareInterface>hardware_interface/PositionJointInterface</hardwareInterface>
             </actuator>
@@ -68,5 +68,5 @@
             <actuator name="front_${prefix}_motor">
                 <mechanicalReduction>1.0</mechanicalReduction>
-                <motorTorqueConstant>1.o</motorTorqueConstant>
+                <motorTorqueConstant>1.0</motorTorqueConstant>
                 <hardwareInterface>hardware_interface/VelocityJointInterface</hardwareInterface>
             </actuator>
@@ -106,5 +106,5 @@
             <actuator name="rear_${prefix}_motor">
                 <mechanicalReduction>1.0</mechanicalReduction>
-                <motorTorqueConstant>1.o</motorTorqueConstant>
+                <motorTorqueConstant>1.0</motorTorqueConstant>
                 <hardwareInterface>hardware_interface/VelocityJointInterface</hardwareInterface>
             </actuator>

Commit message: adding imu_sensor_plugin

File: fellahbot_description/urdf/fellahbot.urdf.xacro (robot description, xacro)
@@ -65,8 +65,30 @@
     <xacro:default_inertial mass="0.2"/>
   </link>
-  <joint name="base_camera" type="fixed">
+  <joint name="base_camera_sensor" type="fixed">
     <parent link="chassis"/>
     <child link="camera"/>
     <origin xyz="0.555 0.0 0.130"/>
+  </joint>
+  <!-- camera link -->
+  <link name="imu_link">
+    <visual>
+      <geometry>
+        <box size="0.06 .03 0.01"/>
+      </geometry>
+      <origin rpy="0 0 0" xyz="0 0 0"/>
+      <material name="blue"/>
+    </visual>
+    <collision>
+      <geometry>
+        <box size="0.06 .03 0.01"/>
+      </geometry>
+    </collision>
+    <xacro:solid_cuboid_inertial rpy="0 0 0" xyz="0.319 0.0 0.130" mass="0.2" x="0.06" y="0.03" z="0.01" />
+    <xacro:default_inertial mass="0.02"/>
+  </link>
+  <joint name="base_imu_sensor" type="fixed">
+    <parent link="chassis"/>
+    <child link="imu_link"/>
+    <origin xyz="0.319 0.0 0.130"/>
   </joint>
   <!-- Lightning -->

File: fellahbot_description/urdf/plugin.gazebo.xacro (robot description, xacro)
@@ -84,5 +84,5 @@
       <topic>imu_data</topic>
       <plugin filename="libgazebo_ros_imu_sensor.so" name="imu_plugin">
-        <topicName>imu</topicName>
+        <topicName>imu_data</topicName>
         <bodyName>imu_link</bodyName>
         <updateRateHZ>10.0</updateRateHZ>

Commit message: solving inertial para causing robot drift position

File: fellahbot_description/urdf/fellahbot.urdf.xacro (robot description, xacro)
@@ -6,4 +6,6 @@
   <xacro:include filename="$(find fellahbot_description)/urdf/plugin.gazebo.xacro"/>
   <xacro:include filename="$(find fellahbot_description)/urdf/wheel.xacro"/>
+  <xacro:include filename="$(find fellahbot_description)/urdf/transmission.xacro"/>
+  <xacro:include filename="$(find fellahbot_description)/urdf/ackermann_controller.xacro"/>
   <link name="base_link"/>
   <!-- Chassis link -->
@@ -18,8 +20,8 @@
     <collision>
       <geometry>
-        <box size="${chassis_length} ${chassis_width} ${chassis_height}"/>
+        <mesh filename="package://fellahbot_description/meshes/Fellahbot_DAE/Parts/ChassisRobot-Fusion001.dae"/>
       </geometry>
     </collision>
-    <xacro:solid_cuboid_inertial rpy="0 0 0" xyz="0.0 0.0 0.359" mass="${chassis_mass}" x="${chassis_length}" y="${chassis_width}" z="0.411" />
+    <xacro:solid_cuboid_inertial rpy="0 0 0" xyz="0.0 0.0 0.0" mass="${chassis_mass}" x="${chassis_length}" y="${chassis_width}" z="0.411" />
   </link>
   <joint name="base_robot" type="fixed">
@@ -27,4 +29,5 @@
     <child link="chassis"/>
     <origin rpy="0 0 0" xyz="0 0 0.359"/>
+    <dynamics damping="0.0" friction="0.0"/>
   </joint>
   <!-- lidar link -->
@@ -41,5 +44,5 @@
       </geometry>
     </collision>
-    <xacro:solid_cylinder_inertial rpy="0 0 0" xyz="0.455 0.0 -0.028" mass="0.3" radius="0.04" length="0.06" />
+    <xacro:solid_cylinder_inertial rpy="0 0 0" xyz="0.0 0.0 0.0" mass="0.3" radius="0.04" length="0.06" />
   </link>
   <joint name="base_lidar" type="fixed">
@@ -47,4 +50,5 @@
     <child link="laser"/>
     <origin xyz="0.455 0.0 -0.028"/>
+    <dynamics damping="0.0" friction="0.0"/>
   </joint>
   <!-- camera link -->
@@ -62,5 +66,5 @@
       </geometry>
     </collision>
-    <xacro:solid_cuboid_inertial rpy="0 0 0" xyz="0.555 0.0 0.130" mass="0.2" x="0.01" y="0.06" z="0.03" />
+    <xacro:solid_cuboid_inertial rpy="0 0 0" xyz="0.0 0.0 0.0" mass="0.2" x="0.01" y="0.06" z="0.03" />
     <xacro:default_inertial mass="0.2"/>
   </link>
@@ -69,4 +73,5 @@
     <child link="camera"/>
     <origin xyz="0.555 0.0 0.130"/>
+    <dynamics damping="0.0" friction="0.0"/>
   </joint>
   <!-- camera link -->
@@ -84,5 +89,5 @@
       </geometry>
     </collision>
-    <xacro:solid_cuboid_inertial rpy="0 0 0" xyz="0.319 0.0 0.130" mass="0.2" x="0.06" y="0.03" z="0.01" />
+    <xacro:solid_cuboid_inertial rpy="0 0 0" xyz="0.0 0.0 0.0" mass="0.02" x="0.06" y="0.03" z="0.01" />
     <xacro:default_inertial mass="0.02"/>
   </link>
@@ -91,4 +96,5 @@
     <child link="imu_link"/>
     <origin xyz="0.319 0.0 0.130"/>
+    <dynamics damping="0.0" friction="0.0"/>
   </joint>
   <!-- Lightning -->
@@ -103,9 +109,9 @@
     <collision>
       <geometry>
-        <cylinder radius="0.03" length="0.3"/>
+        <cylinder radius="0.025" length="0.290"/>
       </geometry>
       <origin rpy="${math_pi_over_2} 0 0" xyz="0 0 0"/>
     </collision>
-    <xacro:solid_cylinder_inertial rpy="0 0 0" xyz="0.556 0.0 0.27444" mass="0.5" radius="0.025" length="0.29" />
+    <xacro:solid_cylinder_inertial rpy="0 0 0" xyz="0.0 0.0 0.0" mass="0.5" radius="0.025" length="0.29" />
   </link>
   <joint name="base_phare" type="fixed">
@@ -113,98 +119,12 @@
     <child link="phare"/>
     <origin xyz="0.556 0.0 0.27444"/>
+    <dynamics damping="0.0" friction="0.0"/>
   </joint>
   <!-- Wheels -->
-  <xacro:front_steer_wheel prefix="left" parent="chassis" reflect="1" />
-  <xacro:front_steer_wheel prefix="right" parent="chassis" reflect="-1" />
-  <xacro:rear_wheel prefix="left" parent="chassis" reflect="1" />
-  <xacro:rear_wheel prefix="right" parent="chassis" reflect="-1" />
+  <xacro:front_steer_wheel prefix="front_left" parent="chassis" reflect="1" />
+  <xacro:front_steer_wheel prefix="front_right" parent="chassis" reflect="-1" />
+  <xacro:rear_wheel prefix="rear_left" parent="chassis" reflect="1" />
+  <xacro:rear_wheel prefix="rear_right" parent="chassis" reflect="-1" />
   <!-- joints for ackermann_steering_controller -->
-  <link name="steer_link">
-    <visual>
-      <origin xyz="0 0 0" rpy="0 0 0"/>
-      <geometry>
-        <cylinder radius="0.05" length="0.03"/>
-      </geometry>
-      <material name="yellow"/>
-    </visual>
-    <collision>
-      <origin xyz="0 0 0" rpy="0 0 0"/>
-      <geometry>
-        <cylinder radius="0.05" length="0.03"/>
-      </geometry>
-      <material name="yellow"/>
-    </collision>
-    <xacro:solid_cylinder_inertial rpy="0 0 0" xyz="0.319 0.0 0.0" mass="6" radius="0.05" length="0.03" />
-  </link>
-  <joint name="steer_joint" type="revolute">
-    <parent link="chassis"/>
-    <child link="steer_link"/>
-    <axis xyz="0 0 1"/>
-    <limit lower="${-math_pi_over_6_29}" upper="${math_pi_over_6}" velocity="50.0" effort="100.0"/>
-    <origin xyz="0.319 0.0 0.0"/>
-  </joint>
-  <!-- Transmission is important to link the joints and the controller -->
-  <transmission name="steer_joint_trans">
-    <type>transmission_interface/SimpleTransmission</type>
-    <actuator name="steer_joint_motor">
-      <mechanicalReduction>1.0</mechanicalReduction>
-      <motorTorqueConstant>1.0</motorTorqueConstant>
-      <hardwareInterface>hardware_interface/PositionJointInterface</hardwareInterface>
-    </actuator>
-    <joint name="steer_joint">
-      <hardwareInterface>hardware_interface/PositionJointInterface</hardwareInterface>
-    </joint>
-  </transmission>
-  <gazebo reference="steer_link">
-    <material>Gazebo/Yellow</material>
-    <mu1 value="1.0"/>
-    <mu2 value="1.0"/>
-    <kp value="10000000.0" />
-    <kd value="1.0" />
-    <fdir1 value="1 0 0"/>
-  </gazebo>
-  <link name="wheel_link">
-    <visual>
-      <origin xyz="0 0 0" rpy="${math_pi_over_2} 0 0"/>
-      <geometry>
-        <cylinder radius="0.03" length="0.05"/>
-      </geometry>
-      <material name="yellow"/>
-    </visual>
-    <collision>
-      <origin xyz="0 0 0" rpy="${math_pi_over_2} 0 0"/>
-      <geometry>
-        <cylinder radius="0.03" length="0.05"/>
-      </geometry>
-      <material name="yellow"/>
-    </collision>
-    <xacro:solid_cylinder_inertial rpy="0 0 0" xyz="-0.335 0.0 -0.192" mass="6" radius="0.03" length="0.05" />
-  </link>
-  <joint name="wheel_joint" type="continuous">
-    <parent link="chassis"/>
-    <child link="wheel_link"/>
-    <origin xyz="-0.335 0.0 -0.192" rpy="0 0 0"/>
-    <limit effort="150" velocity="20"/>
-    <joint_properties damping="1.0" friction="1.0"/>
-  </joint>
-  <!-- Transmission is important to link the joints and the controller -->
-  <transmission name="wheel_transmission">
-    <type>transmission_interface/SimpleTransmission</type>
-    <joint name="wheel_joint">
-      <hardwareInterface>hardware_interface/VelocityJointInterface</hardwareInterface>
-    </joint>
-    <actuator name="wheel_joint_motor">
-      <mechanicalReduction>1.0</mechanicalReduction>
-      <motorTorqueConstant>1.0</motorTorqueConstant>
-      <hardwareInterface>hardware_interface/VelocityJointInterface</hardwareInterface>
-    </actuator>
-  </transmission>
-  <gazebo reference="wheel_link">
-    <material>Gazebo/Yellow</material>
-    <mu1 value="1.0"/>
-    <mu2 value="1.0"/>
-    <kp value="10000000.0" />
-    <kd value="1.0" />
-    <fdir1 value="1 0 0"/>
-  </gazebo>
+  <xacro:ackermann_steering_controller prefix="ackermann" parent="chassis" />
 </robot>
