Commit message: add inertial correction and transmission macro

File: fellahbot_description/urdf/wheel.xacro (robot description, xacro)
@@ -3,9 +3,7 @@
     <xacro:include filename="$(find fellahbot_description)/urdf/constants.xacro"/>
     <xacro:include filename="$(find fellahbot_description)/urdf/inertials.xacro"/>
+    <xacro:include filename="$(find fellahbot_description)/urdf/transmission.xacro"/>
     <xacro:macro name="front_steer_wheel" params="prefix parent reflect ">
-        <xacro:property name="pos_x_joint" value="${((chassis_length / 2)- wheel_radius)}"/>
-        <xacro:property name="pos_y_joint" value="${((chassis_width / 2) - (wheel_width / 2))}"/>
-        <xacro:property name="pos_z_joint" value="-${chassis_to_ground - wheel_radius}"/>
-        <link name="front_${prefix}_steer">
+        <link name="${prefix}_steer">
             <visual>
                 <geometry>
@@ -19,25 +17,16 @@
                 </geometry>
             </collision>
-            <xacro:default_inertial mass="6"/>
+            <xacro:solid_cylinder_inertial rpy="0 0 0" xyz="0.0 0.0 0.0" mass="6" radius="0.085" length="0.215" />
         </link>
-        <joint name="front_${prefix}_steer_joint" type="revolute">
+        <joint name="${prefix}_steer_joint" type="revolute">
             <parent link="${parent}"/>
-            <child link="front_${prefix}_steer"/>
+            <child link="${prefix}_steer"/>
             <axis xyz="0 0 1"/>
-            <limit lower="${-math_pi_over_6_29}" upper="${math_pi_over_6}" velocity="50.0" effort="100"/>
+            <limit lower="${-1.0 * math_pi_over_6}" upper="${math_pi_over_6}" velocity="5.0" effort="100"/>
             <origin xyz="0.319 ${(reflect * 0.175)} 0.0"/>
+            <dynamics damping="0.7" friction="0.7"/>
         </joint>
-        <transmission name="front_${prefix}_steer_transmission">
-            <type>transmission_interface/SimpleTransmission</type>
-            <joint name="front_${prefix}_steer_joint">
-                <hardwareInterface>hardware_interface/PositionJointInterface</hardwareInterface>
-            </joint>
-            <actuator name="front_${prefix}_steer_motor">
-                <mechanicalReduction>1.0</mechanicalReduction>
-                <motorTorqueConstant>1.0</motorTorqueConstant>
-                <hardwareInterface>hardware_interface/PositionJointInterface</hardwareInterface>
-            </actuator>
-        </transmission>
-        <link name="front_${prefix}_wheel">
+        <xacro:transmission_steer prefix="${prefix}" />
+        <link name="${prefix}_wheel">
             <visual>
                 <geometry>
@@ -51,38 +40,22 @@
                 </geometry>
             </collision>
-            <xacro:solid_cylinder_inertial rpy="0 0 0" xyz="0.0 0.0 -0.192" mass="${wheel_mass}" radius="${wheel_radius}" length="${wheel_width}" />
+            <xacro:solid_cylinder_inertial rpy="0 0 0" xyz="0.0 0.0 0.0" mass="${wheel_mass}" radius="${wheel_radius}" length="${wheel_width}" />
         </link>
-        <joint name="front_${prefix}_wheel_joint" type="continuous">
-            <parent link="front_${prefix}_steer"/>
-            <child link="front_${prefix}_wheel"/>
+        <joint name="${prefix}_wheel_joint" type="continuous">
+            <parent link="${prefix}_steer"/>
+            <child link="${prefix}_wheel"/>
             <axis xyz="0 1 0"/>
             <origin xyz="0.0 0.0 -0.192" rpy="0 0 0"/>
             <limit effort="150" velocity="20"/>
-            <joint_properties damping="1.0" friction="1.0"/>
+            <dynamics damping="0.7" friction="0.7"/>
         </joint>
-        <transmission name="front_${prefix}_wheel_transmission">
-            <type>transmission_interface/SimpleTransmission</type>
-            <joint name="front_${prefix}_wheel_joint">
-                <hardwareInterface>hardware_interface/VelocityJointInterface</hardwareInterface>
-            </joint>
-            <actuator name="front_${prefix}_motor">
-                <mechanicalReduction>1.0</mechanicalReduction>
-                <motorTorqueConstant>1.0</motorTorqueConstant>
-                <hardwareInterface>hardware_interface/VelocityJointInterface</hardwareInterface>
-            </actuator>
-        </transmission>
-        <gazebo reference="front_${prefix}_wheel">
-            <mu1 value="1.0"/>
-			<mu2 value="1.0"/>
-			<kp value="10000000.0" />
-			<kd value="1.0" />
-			<fdir1 value="1 0 0"/>
+        <xacro:transmission_wheel prefix="${prefix}" />
+        <gazebo reference="${prefix}_wheel">
+            <mu1 value="1.6"/>
+			<mu2 value="1.6"/>
         </gazebo>
     </xacro:macro>
     <xacro:macro name="rear_wheel" params="prefix parent reflect ">
-        <xacro:property name="pos_x_joint" value="${((chassis_length / 2)- wheel_radius)}"/>
-        <xacro:property name="pos_y_joint" value="${((chassis_width / 2) - (wheel_width / 2))}"/>
-        <xacro:property name="pos_z_joint" value="-${chassis_to_ground - wheel_radius}"/>
-        <link name="rear_${prefix}_wheel">
+        <link name="${prefix}_wheel">
             <visual>
                 <geometry>
@@ -96,31 +69,18 @@
                 </geometry>
             </collision>
-            <xacro:solid_cylinder_inertial rpy="0 0 0" xyz="-0.335 ${(reflect * 0.17523)} -0.192" mass="${wheel_mass}" radius="${wheel_radius}" length="${wheel_width}" />
+            <xacro:solid_cylinder_inertial rpy="0 0 0" xyz="0.0 0.0 0.0" mass="${wheel_mass}" radius="${wheel_radius}" length="${wheel_width}" />
         </link>
-        <joint name="rear_${prefix}_wheel_joint" type="continuous">
+        <joint name="${prefix}_wheel_joint" type="continuous">
             <parent link="${parent}"/>
-            <child link="rear_${prefix}_wheel"/>
+            <child link="${prefix}_wheel"/>
             <axis xyz="0 1 0"/>
             <origin xyz="-0.335 ${(reflect * 0.17523)} -0.192" rpy="0 0 0"/>
             <limit effort="150" velocity="20"/>
-            <joint_properties damping="1.0" friction="1.0"/>
+            <dynamics damping="0.7" friction="0.7"/>
         </joint>
-        <transmission name="rear_${prefix}_wheel_transmission">
-            <type>transmission_interface/SimpleTransmission</type>
-            <joint name="rear_${prefix}_wheel_joint">
-                <hardwareInterface>hardware_interface/VelocityJointInterface</hardwareInterface>
-            </joint>
-            <actuator name="rear_${prefix}_motor">
-                <mechanicalReduction>1.0</mechanicalReduction>
-                <motorTorqueConstant>1.0</motorTorqueConstant>
-                <hardwareInterface>hardware_interface/VelocityJointInterface</hardwareInterface>
-            </actuator>
-        </transmission>
-        <gazebo reference="rear_${prefix}_wheel">
-            <mu1 value="1.0"/>
-			<mu2 value="1.0"/>
-			<kp value="10000000.0" />
-			<kd value="1.0" />
-			<fdir1 value="1 0 0"/>
+        <xacro:transmission_wheel prefix="${prefix}" />
+        <gazebo reference="${prefix}_wheel">
+            <mu1 value="1.6"/>
+			<mu2 value="1.6"/>
         </gazebo>
     </xacro:macro>
