Commit message: gazebo inertial correction

File: fellahbot_description/urdf/ackermann_controller.xacro (robot description, xacro)
@@ -32,4 +32,9 @@
         </joint>
         <xacro:transmission_steer prefix="${prefix}" />
+        <gazebo reference="${prefix}_steer_link">
+            <material>Gazebo/Yellow</material>
+            <mu1 value="1.6"/>
+            <mu2 value="1.6"/>
+        </gazebo>
         <!-- joints for ackermann_speed_controller -->
         <link name="${prefix}_wheel_link">
@@ -48,5 +53,5 @@
                 <material name="yellow"/>
             </collision>
-            <xacro:solid_cylinder_inertial rpy="0 0 0" xyz="0.0 0.0 0.0" mass="6" radius="0.03" length="0.05" />
+            <xacro:solid_cylinder_inertial rpy="${math_pi_over_2} 0 0" xyz="0.0 0.0 0.0" mass="6" radius="0.03" length="0.05" />
         </link>
         <joint name="${prefix}_wheel_joint" type="continuous">
@@ -65,3 +70,27 @@
         </gazebo>
     </xacro:macro>
+    <xacro:macro name="ackermann_steering_controller_link" params="prefix parent ">
+        <!-- joints for ackermann_steer_controller -->
+        <link name="${prefix}_steer_link"/>
+        <joint name="${prefix}_steer_joint" type="revolute">
+            <parent link="${parent}"/>
+            <child link="${prefix}_steer_link"/>
+            <axis xyz="0 0 1"/>
+            <limit lower="${-1.0 * math_pi_over_6}" upper="${math_pi_over_6}" velocity="5.0" effort="100.0"/>
+            <origin xyz="0.319 0.0 0.0"/>
+            <dynamics damping="0.7" friction="0.7"/>
+        </joint>
+        <xacro:transmission_steer prefix="${prefix}" />
+        <!-- joints for ackermann_speed_controller -->
+        <link name="${prefix}_wheel_link"/>
+        <joint name="${prefix}_wheel_joint" type="continuous">
+            <parent link="${parent}"/>
+            <child link="${prefix}_wheel_link"/>
+            <axis xyz="0 1 0"/>
+            <origin xyz="-0.335 0.0 -0.192" rpy="0 0 0"/>
+            <limit effort="150" velocity="20"/>
+            <dynamics damping="0.7" friction="0.7"/>
+        </joint>
+        <xacro:transmission_wheel prefix="${prefix}" />
+    </xacro:macro>
 </robot>

File: fellahbot_description/urdf/constants.xacro (robot description, xacro)
@@ -10,17 +10,18 @@
 	<!-- Chassis properties -->
 	<xacro:property name="chassis_height" value="0.311"/>
+	<xacro:property name="chassis_height_v2" value="${(robot_height_truth_ground - (wheel_radius))}"/>
 	<!--xacro:property name="chassis_height" value="0.470"/-->
 	<!--xacro:property name="chassis_height" value="0.411"/-->
 	<xacro:property name="chassis_length" value="1.150"/>
 	<xacro:property name="chassis_width" value="0.632"/>
-	<xacro:property name="chassis_mass" value="100.00"/>
+	<xacro:property name="chassis_mass" value="80.00"/>
 	<xacro:property name="robot_height_truth_ground" value="0.632"/>
 	<xacro:property name="chassis_to_ground" value="${(robot_height_truth_ground - (chassis_height/2))}"/>
 	<!-- Caster wheel properties -->
 	<xacro:property name="caster_radius" value="0.020"/>
-	<xacro:property name="caster_mass" value="0.09"/>
+	<xacro:property name="caster_mass" value="6.0"/>
 	<xacro:property name="caster_offsetX" value="0.045"/>
 	<!-- 13" geared Wheels properties -->
-	<xacro:property name="wheel_width" value="0.105"/>
+	<xacro:property name="wheel_width" value="0.135"/>
 	<xacro:property name="wheel_radius" value="0.167"/>
 	<xacro:property name="wheel_diameters" value="0.334"/>

File: fellahbot_description/urdf/fellahbot.urdf.xacro (robot description, xacro)
@@ -23,5 +23,5 @@
       </geometry>
     </collision>
-    <xacro:solid_cuboid_inertial rpy="0 0 0" xyz="0.0 0.0 0.0" mass="${chassis_mass}" x="${chassis_length}" y="${chassis_width}" z="0.411" />
+    <xacro:solid_cuboid_inertial rpy="0 0 0" xyz="0.0 0.0 0.0" mass="${chassis_mass}" x="${chassis_length}" y="${chassis_width}" z="${chassis_height_v2}" />
   </link>
   <joint name="base_robot" type="fixed">
@@ -127,4 +127,4 @@
   <xacro:rear_wheel prefix="rear_right" parent="chassis" reflect="-1" />
   <!-- joints for ackermann_steering_controller -->
-  <xacro:ackermann_steering_controller prefix="ackermann" parent="chassis" />
+  <xacro:ackermann_steering_controller_link prefix="ackermann" parent="chassis" />
 </robot>

File: fellahbot_description/urdf/wheel.xacro (robot description, xacro)
@@ -40,5 +40,5 @@
                 </geometry>
             </collision>
-            <xacro:solid_cylinder_inertial rpy="0 0 0" xyz="0.0 0.0 0.0" mass="${wheel_mass}" radius="${wheel_radius}" length="${wheel_width}" />
+            <xacro:solid_cylinder_inertial rpy="${math_pi_over_2} 0 0" xyz="0.0 0.0 0.0" mass="${wheel_mass}" radius="${wheel_radius}" length="${wheel_width}" />
         </link>
         <joint name="${prefix}_wheel_joint" type="continuous">
@@ -69,5 +69,5 @@
                 </geometry>
             </collision>
-            <xacro:solid_cylinder_inertial rpy="0 0 0" xyz="0.0 0.0 0.0" mass="${wheel_mass}" radius="${wheel_radius}" length="${wheel_width}" />
+            <xacro:solid_cylinder_inertial rpy="${math_pi_over_2} 0 0" xyz="0.0 0.0 0.0" mass="${wheel_mass}" radius="${wheel_radius}" length="${wheel_width}" />
         </link>
         <joint name="${prefix}_wheel_joint" type="continuous">
